File: Mega_Shield/Mega_Shield.kicad_sch (KiCad schematic)
At the start: 2 parts, among them J1 DE9_Socket_MountingHoles

Commit message: Added in some pins
Connections:
- net GND: now reaches J1.1
- net GND: now also J1.6, J1.SH (PAD)
- net PWM_PIN_1: now reaches J1.2
- net SENSOR_PIN_1: now reaches J1.3
- net +12V: now reaches J1.4
- net +12V: now also J1.5, J1.9
- net LIMIT_PIN_1: now reaches J1.7
- net LED_PIN_1: now reaches J1.8

Commit message: updates
Parts:
- added J10, J11, J12, J2, J3, J4, J5, J6, J7, J8, J9: DE9_Socket_MountingHoles, mega_shield_footprint:61800929321, symbol Connector:DE9_Socket_MountingHoles
- added J13: Conn_01x02, symbol Connector_Generic:Conn_01x02
- J1: footprint mega_shield_footprint:ASSMANN_A-DF_09_A_KG-T2S -> mega_shield_footprint:61800929321
Connections:
- net +12V: now also U1.VIN, J10.4, J10.5, J10.9, J11.4, J11.5, J11.9, J12.4, J12.5, J12.9, J13.1 (Pin_1), J2.4, J2.5, J2.9, J3.4, J3.5, J3.9, J4.4, J4.5, J4.9, J5.4, J5.5, J5.9, J6.4, J6.5, J6.9, J7.4, J7.5, J7.9, J8.4, J8.5, J8.9, J9.4, J9.5, J9.9
- net GND: now also U1.GND1, U1.GND2, U1.GND3, U1.GND4, U1.GND5, J10.1, J10.6, J10.SH (PAD), J11.1, J11.6, J11.SH (PAD), J12.1, J12.6, J12.SH (PAD), J13.2 (Pin_2), J2.1, J2.6, J2.SH (PAD), J3.1, J3.6, J3.SH (PAD), J4.1, J4.6, J4.SH (PAD), J5.1, J5.6, J5.SH (PAD), J6.1, J6.6, J6.SH (PAD), J7.1, J7.6, J7.SH (PAD), J8.1, J8.6, J8.SH (PAD), J9.1, J9.6, J9.SH (PAD)
- net LED_PIN_1: now also J9.8; no longer J1.8
- net LIMIT_PIN_1: now also J9.7; no longer J1.7
- net PWM_PIN_1: now also U1.2, J9.2; no longer J1.2
- net PWM_PIN_12: now also U1.13, J5.2
- net SENSOR_PIN_1: now also J9.3; no longer J1.3
- net PWM_PIN_9: now reaches U1.10
- net PWM_PIN_9: now also J11.2
- net PWM_PIN_10: now reaches U1.11
- net PWM_PIN_10: now also J6.2
- net PWM_PIN_11: now reaches U1.12
- net PWM_PIN_11: now also J4.2
- net PWM_PIN_2: now reaches U1.3
- net PWM_PIN_2: now also J7.2
- net PWM_PIN_3: now reaches U1.4
- net PWM_PIN_3: now also J8.2
- net PWM_PIN_4: now reaches U1.5
- net PWM_PIN_4: now also J1.2
- net PWM_PIN_5: now reaches U1.6
- net PWM_PIN_5: now also J2.2
- net PWM_PIN_6: now reaches U1.7
- net PWM_PIN_6: now also J3.2
- net PWM_PIN_7: now reaches U1.8
- net PWM_PIN_7: now also J12.2
- net PWM_PIN_8: now reaches U1.9
- net PWM_PIN_8: now also J10.2
- new net LED_PIN_10: J6.8
- new net LED_PIN_11: J4.8
- new net LED_PIN_12: J5.8
- new net LED_PIN_2: J7.8
- new net LED_PIN_3: J8.8
- new net LED_PIN_4: J1.8
- new net LED_PIN_5: J2.8
- new net LED_PIN_6: J3.8
- new net LED_PIN_7: J12.8
- new net LED_PIN_8: J10.8
- new net LED_PIN_9: J11.8
- new net LIMIT_PIN_10: J6.7
- new net LIMIT_PIN_11: J4.7
- new net LIMIT_PIN_12: J5.7
- new net LIMIT_PIN_2: J7.7
- new net LIMIT_PIN_3: J8.7
- new net LIMIT_PIN_4: J1.7
- new net LIMIT_PIN_5: J2.7
- new net LIMIT_PIN_6: J3.7
- new net LIMIT_PIN_7: J12.7
- new net LIMIT_PIN_8: J10.7
- new net LIMIT_PIN_9: J11.7
- new net SENSOR_PIN_10: J6.3
- new net SENSOR_PIN_11: J4.3
- new net SENSOR_PIN_12: J5.3
- new net SENSOR_PIN_2: J7.3
- new net SENSOR_PIN_3: J8.3
- new net SENSOR_PIN_4: J1.3
- new net SENSOR_PIN_5: J2.3
- new net SENSOR_PIN_6: J3.3
- new net SENSOR_PIN_7: J12.3
- new net SENSOR_PIN_8: J10.3
- new net SENSOR_PIN_9: J11.3
Other:
- moved on the sheet: J1, U1

Commit message: Finished Mega shield
Parts:
- added C1: 220uF, Capacitor_SMD:CP_Elec_8x10, symbol Device:C_Polarized_US
- added D1: PWR, LED_SMD:LED_0805_2012Metric, symbol Device:LED
- added J14: Serial, mega_shield_footprint:TE_640457-3, symbol Connector_Generic:Conn_01x03
- added R1: 5.23k, Fan_Blower_PCB:R0805, symbol Device:R_US
- J13: value Conn_01x02 -> PWR IN; footprint (none) -> mega_shield_footprint:TE_640389-2; Distributor (none) -> Digikey; Distributor PN (none) -> A1976-ND; Mfg. (none) -> TE Connectivity AMP Connectors; Mfg. PN (none) -> 640389-2
- U1: value (none) -> Arduino Mega
Connections:
- net +12V: now also C1.1, R1.1
- net GND: now also C1.2, D1.1 (K), J14.1 (Pin_1)
- net LED_PIN_1: now also U1.15
- net LED_PIN_10: now also U1.41
- net LED_PIN_11: now also U1.47
- net LED_PIN_12: now also U1.53
- net LED_PIN_2: now also U1.24
- net LED_PIN_3: now also U1.30
- net LED_PIN_4: now also U1.36
- net LED_PIN_5: now also U1.42
- net LED_PIN_6: now also U1.48
- net LED_PIN_7: now also U1.23
- net LED_PIN_8: now also U1.29
- net LED_PIN_9: now also U1.35
- net LIMIT_PIN_1: now also U1.17
- net LIMIT_PIN_10: now also U1.37
- net LIMIT_PIN_11: now also U1.43
- net LIMIT_PIN_12: now also U1.49
- net LIMIT_PIN_2: now also U1.14
- net LIMIT_PIN_3: now also U1.26
- net LIMIT_PIN_4: now also U1.32
- net LIMIT_PIN_5: now also U1.38
- net LIMIT_PIN_6: now also U1.44
- net LIMIT_PIN_7: now also U1.50
- net LIMIT_PIN_8: now also U1.25
- net LIMIT_PIN_9: now also U1.31
- net SENSOR_PIN_1: now also U1.16
- net SENSOR_PIN_10: now also U1.39
- net SENSOR_PIN_11: now also U1.45
- net SENSOR_PIN_12: now also U1.51
- net SENSOR_PIN_2: now also U1.22
- net SENSOR_PIN_3: now also U1.28
- net SENSOR_PIN_4: now also U1.34
- net SENSOR_PIN_5: now also U1.40
- net SENSOR_PIN_6: now also U1.46
- net SENSOR_PIN_7: now also U1.52
- net SENSOR_PIN_8: now also U1.27
- net SENSOR_PIN_9: now also U1.33
- net Tx: now reaches U1.18
- net Tx: now also J14.3 (Pin_3)
- net Rx: now reaches U1.19
- net Rx: now also J14.2 (Pin_2)
- new net: D1.2 (A), R1.2
- no-connect marks 0 -> 30

Commit message: board layout
Parts:
- J10, J11: Distributor PN AE10921-ND -> 732-61800929321-ND; Mfg. Assmann WSW Components -> Würth Elektronik; Mfg. PN A-DF 09 A/KG-T2S -> 61800929321
- J12: renamed from J6; Distributor PN AE10921-ND -> 732-61800929321-ND; Mfg. Assmann WSW Components -> Würth Elektronik; Mfg. PN A-DF 09 A/KG-T2S -> 61800929321
- J13: renamed from J4; Distributor Digikey -> Würth Elektronik; Distributor PN AE10921-ND -> 732-61800929321-ND; Mfg. Assmann WSW Components -> Würth Elektronik; Mfg. PN A-DF 09 A/KG-T2S -> 61800929321
- J14: renamed from J5; Distributor PN AE10921-ND -> 732-61800929321-ND; Mfg. Assmann WSW Components -> Würth Elektronik; Mfg. PN A-DF 09 A/KG-T2S -> 61800929321
- J3: renamed from J9; Distributor PN AE10921-ND -> 732-61800929321-ND; Mfg. Assmann WSW Components -> Würth Elektronik; Mfg. PN A-DF 09 A/KG-T2S -> Würth Elektronik
- J4: renamed from J7; Distributor PN AE10921-ND -> 732-61800929321-ND; Mfg. Assmann WSW Components -> Würth Elektronik; Mfg. PN A-DF 09 A/KG-T2S -> 61800929321
- J5: renamed from J8; Distributor PN AE10921-ND -> 732-61800929321-ND; Mfg. Assmann WSW Components -> Würth Elektronik; Mfg. PN A-DF 09 A/KG-T2S -> 61800929321
- J6: renamed from J1; Distributor PN AE10921-ND -> 732-61800929321-ND; Mfg. Assmann WSW Components -> Würth Elektronik; Mfg. PN A-DF 09 A/KG-T2S -> 61800929321
- J7: renamed from J2; Distributor PN AE10921-ND -> 732-61800929321-ND; Mfg. Assmann WSW Components -> Würth Elektronik; Mfg. PN A-DF 09 A/KG-T2S -> 61800929321
- J8: renamed from J3; Distributor PN AE10921-ND -> 732-61800929321-ND; Mfg. Assmann WSW Components -> Würth Elektronik; Mfg. PN A-DF 09 A/KG-T2S -> 61800929321
- J9: renamed from J12; Distributor PN AE10921-ND -> 732-61800929321-ND; Mfg. Assmann WSW Components -> Würth Elektronik; Mfg. PN A-DF 09 A/KG-T2S -> 61800929321
- R1: footprint Fan_Blower_PCB:R0805 -> Resistor_SMD:R_0805_2012Metric
- renumbered J13 to J1, J14 to J2
Other:
- moved on the sheet: J10, J11, J13, J14, J4, J5, J7, J8
