File: Mega_Shield/Mega_Shield.kicad_pcb (KiCad board)
At the start: 2 copper layers, 18 parts, among them J1 DE9_Socket_MountingHoles, J10 DE9_Socket_MountingHoles, J11 DE9_Socket_MountingHoles, J12 DE9_Socket_MountingHoles, J13 PWR IN, J14 Serial, J2 DE9_Socket_MountingHoles, J3 DE9_Socket_MountingHoles, J4 DE9_Socket_MountingHoles, J5 DE9_Socket_MountingHoles, J6 DE9_Socket_MountingHoles, J7 DE9_Socket_MountingHoles, J8 DE9_Socket_MountingHoles, J9 DE9_Socket_MountingHoles, U1 Arduino Mega

Commit message: Board layout updates
Parts:
- moved J14 353.2 mm to (262.7, 105.7), turned to -90 degrees
- moved J13 351.2 mm to (262.7, 67.6), turned to -90 degrees
- moved J11 335.5 mm to (237.3, 67.6), turned to -90 degrees
- moved J12 326.5 mm to (237.3, 105.7), turned to -90 degrees
- moved J9 314.9 mm to (211.9, 67.6), turned to -90 degrees
- moved J10 301.4 mm to (211.9, 105.7), turned to -90 degrees
- moved J8 283.4 mm to (186.5, 105.7), turned to -90 degrees
- moved J7 278.5 mm to (186.5, 67.6), turned to -90 degrees
- moved J6 268.0 mm to (161.1, 105.7), turned to -90 degrees
- moved J5 252.2 mm to (161.1, 67.6), turned to -90 degrees
- moved J3 230.0 mm to (135.7, 67.6), turned to -90 degrees
- moved J4 224.1 mm to (135.7, 105.7), turned to -90 degrees
- moved C1 88.9 mm to (47.3, 124.5)
- moved D1 88.9 mm to (37.3, 132.2)
- moved R1 88.9 mm to (32.9, 132.2)
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- renumbered J13 to J1, J6 to J12, J4 to J13, J5 to J14, J14 to J2, J9 to J3, J7 to J4, J8 to J5, J1 to J6, J2 to J7, J3 to J8, J12 to J9

Commit message: Starting board routing
Routing:
- net PWM_PIN_1: track 0.00 -> 61.4 mm, vias 0 -> 1
- net SENSOR_PIN_1: track 0.00 -> 45.9 mm
- net LED_PIN_1: track 0.00 -> 45.3 mm
- net LIMIT_PIN_1: track 0.00 -> 40.7 mm
Changed lines of the file:
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@@
 		)
+	)
+	(segment
+		(start 105.41 60.96)
+		(end 104.648 61.722)
+		(width 0.2)
+		(layer "F.Cu")
+		(net "PWM_PIN_1")
+	)
+	(segment
+		(start 128.778 60.96)
+		(end 105.41 60.96)
+		(width 0.2)
+		(layer "F.Cu")
+		(net "PWM_PIN_1")
+	)
+	(segment
+		(start 130.048 62.23)
+		(end 128.778 60.96)
+		(width 0.2)
+		(layer "F.Cu")
+		(net "PWM_PIN_1")
+	)
+	(segment
+		(start 137.16014 70.35822)
+		(end 133.85822 70.35822)
+		(width 0.2)
+		(layer "F.Cu")
+		(net "PWM_PIN_1")
+	)
+	(segment
+		(start 130.048 66.548)
+		(end 130.048 62.23)
+		(width 0.2)
+		(layer "F.Cu")
+		(net "PWM_PIN_1")
+	)
+	(segment
+		(start 133.85822 70.35822)
+		(end 130.048 66.548)
+		(width 0.2)
+		(layer "F.Cu")
+		(net "PWM_PIN_1")
+	)
+	(via
+		(at 104.648 61.722)
+		(size 0.6)
+		(drill 0.3)
+		(layers "F.Cu" "B.Cu")
+		(net "PWM_PIN_1")
+	)
+	(segment
+		(start 85.18236 61.722)
+		(end 83.28914 63.61522)
+		(width 0.2)
+		(layer "B.Cu")
+		(net "PWM_PIN_1")
+	)
+	(segment
+		(start 104.648 61.722)
+		(end 85.18236 61.722)
+		(width 0.2)
+		(layer "B.Cu")
+		(net "PWM_PIN_1")
+	)
+	(segment
+		(start 131.464 64.985708)
+		(end 131.464 60.482628)
+		(width 0.2)
+		(layer "F.Cu")
+		(net "LED_PIN_1")
+	)
+	(segment
+		(start 101.888675 59.69)
+		(end 99.91436 59.69)
+		(width 0.2)
+		(layer "F.Cu")
+		(net "LED_PIN_1")
+	)
+	(segment
+		(start 130.633372 59.652)
+		(end 101.926674 59.652)
+		(width 0.2)
+		(layer "F.Cu")
+		(net "LED_PIN_1")
+	)
+	(segment
+		(start 101.926674 59.652)
+		(end 101.888675 59.69)
+		(width 0.2)
+		(layer "F.Cu")
+		(net "LED_PIN_1")
+	)
+	(segment
+		(start 134.32014 66.20322)
+		(end 132.681512 66.20322)
+		(width 0.2)
+		(layer "F.Cu")
+		(net "LED_PIN_1")
+	)
+	(segment
+		(start 99.91436 59.69)
+		(end 95.98914 63.61522)
+		(width 0.2)
+		(layer "F.Cu")
+		(net "LED_PIN_1")
+	)
+	(segment
+		(start 132.681512 66.20322)
+		(end 131.464 64.985708)
+		(width 0.2)
+		(layer "F.Cu")
+		(net "LED_PIN_1")
+	)
+	(segment
+		(start 131.464 60.482628)
+		(end 130.633372 59.652)
+		(width 0.2)
+		(layer "F.Cu")
+		(net "LED_PIN_1")
+	)
+	(segment
+		(start 131.064 65.151394)
+		(end 133.500826 67.58822)
+		(width 0.2)
+		(layer "F.Cu")
+		(net "SENSOR_PIN_1")
+	)
+	(segment
+		(start 131.064 60.648314)
+		(end 131.064 65.151394)
+		(width 0.2)
+		(layer "F.Cu")
+		(net "SENSOR_PIN_1")
+	)
+	(segment
+		(start 130.467686 60.052)
+		(end 131.064 60.648314)
+		(width 0.2)
+		(layer "F.Cu")
+		(net "SENSOR_PIN_1")
+	)
+	(segment
+		(start 133.500826 67.58822)
+		(end 137.16014 67.58822)
+		(width 0.2)
+		(layer "F.Cu")
+		(net "SENSOR_PIN_1")
+	)
+	(segment
+		(start 98.52914 63.61522)
+		(end 102.09236 60.052)
+		(width 0.2)
+		(layer "F.Cu")
+		(net "SENSOR_PIN_1")
+	)
+	(segment
+		(start 102.09236 60.052)
+		(end 130.467686 60.052)
+		(width 0.2)
+		(layer "F.Cu")
+		(net "SENSOR_PIN_1")
+	)
+	(segment
+		(start 130.556 60.706)
+		(end 130.302 60.452)
+		(width 0.2)
+		(layer "F.Cu")
+		(net "LIMIT_PIN_1")
+	)
+	(segment
+		(start 134.32014 68.97322)
+		(end 130.556 65.20908)
+		(width 0.2)
+		(layer "F.Cu")
+		(net "LIMIT_PIN_1")
+	)
+	(segment
+		(start 104.23236 60.452)
+		(end 101.06914 63.61522)
+		(width 0.2)
+		(layer "F.Cu")
+		(net "LIMIT_PIN_1")
+	)
+	(segment
+		(start 130.302 60.452)
+		(end 104.23236 60.452)
+		(width 0.2)
+		(layer "F.Cu")
+		(net "LIMIT_PIN_1")
+	)
+	(segment
+		(start 130.556 65.20908)
+		(end 130.556 60.706)
+		(width 0.2)
+		(layer "F.Cu")
+		(net "LIMIT_PIN_1")
 	)
 	(embedded_fonts no)

Commit message: Beginning layout of the single blower
Routing:
- net +12V: track 0.00 -> 389.7 mm
- net PWM_PIN_12: track 0.00 -> 263.7 mm, vias 0 -> 2
- net PWM_PIN_10: track 0.00 -> 236.3 mm
- net PWM_PIN_11: track 0.00 -> 222.1 mm
- net PWM_PIN_8: track 0.00 -> 205.8 mm
- net PWM_PIN_9: track 0.00 -> 193.0 mm
- net SENSOR_PIN_8: track 0.00 -> 175.1 mm, vias 0 -> 3
- net PWM_PIN_6: track 0.00 -> 173.0 mm
- net SENSOR_PIN_12: track 0.00 -> 170.1 mm, vias 0 -> 2
- net LIMIT_PIN_12: track 0.00 -> 165.0 mm
- net SENSOR_PIN_11: track 0.00 -> 163.3 mm, vias 0 -> 1
- net PWM_PIN_7: track 0.00 -> 162.3 mm
- net LED_PIN_11: track 0.00 -> 161.5 mm
- net LED_PIN_12: track 0.00 -> 160.1 mm
- net LIMIT_PIN_11: track 0.00 -> 158.3 mm, vias 0 -> 1
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- added copper zone on B.Cu, net +12V
- added copper zone on B.Cu, net GND
- added copper zone on F.Cu, net GND
Other:
- board outline added: 246.6 x 89.2 mm
- board text added: "+"
- board text added: "-"
- board text added: "GND"
- board text added: "PWR IN"
- board text added: "RX"
- board text added: "TX"

Commit message: Finished routing single blower
Parts:
- moved J13 94.6 mm to (189.6, 127.6), turned to 0 degrees
- moved J14 87.1 mm to (189.6, 153.0), turned to 0 degrees
- moved J7 69.5 mm to (151.5, 127.6), turned to 0 degrees
- moved J8 58.9 mm to (151.5, 153.0), turned to 0 degrees
- moved J10 58.7 mm to (189.6, 51.4), turned to 0 degrees
- moved J4 56.5 mm to (151.5, 51.4), turned to 0 degrees
- moved J11 48.6 mm to (189.6, 76.8), turned to 0 degrees
- moved J12 47.9 mm to (189.6, 102.2), turned to 0 degrees
- moved J9 47.2 mm to (189.6, 26.0), turned to 0 degrees
- moved J3 44.5 mm to (151.5, 26.0), turned to 0 degrees
- moved J5 13.4 mm to (151.5, 76.8), turned to 0 degrees
- moved J6 10.3 mm to (151.5, 102.2), turned to 0 degrees
Routing:
- net +12V: track 389.7 -> 29.2 mm
- net PWM_PIN_12: track 263.7 -> 0.00 mm, vias 2 -> 0
- net PWM_PIN_10: track 236.3 -> 0.00 mm
- net PWM_PIN_11: track 222.1 -> 0.00 mm
- net PWM_PIN_8: track 205.8 -> 0.00 mm
- net PWM_PIN_9: track 193.0 -> 0.00 mm
- net SENSOR_PIN_8: track 175.1 -> 0.00 mm, vias 3 -> 0
- net PWM_PIN_6: track 173.0 -> 0.00 mm
- net SENSOR_PIN_12: track 170.1 -> 0.00 mm, vias 2 -> 0
- net LIMIT_PIN_12: track 165.0 -> 0.00 mm
- net SENSOR_PIN_11: track 163.3 -> 0.00 mm, vias 1 -> 0
- net PWM_PIN_7: track 162.3 -> 0.00 mm
- net LED_PIN_11: track 161.5 -> 0.00 mm
- net LED_PIN_12: track 160.1 -> 0.00 mm
- net LIMIT_PIN_11: track 158.3 -> 0.00 mm, vias 1 -> 0
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Other:
- board size 246.6 x 89.2 mm -> 191.3 x 144.8 mm
